Commit message: fixed sensor placement

File: iiwa_workcell_description/robots/iiwa_workcell.urdf.xacro (robot description, xacro)
@@ -20,5 +20,5 @@
     </xacro:sensor>
     <xacro:sensor parent="$(arg robot_name)_link_2" child="sensor_2_left">
-        <origin xyz="0 0.20 -0.08" rpy="0 ${PI / 2} ${PI / 2}" />
+        <origin xyz="0 0.20 0.08" rpy="0 ${-PI / 2} ${-PI / 2}" />
     </xacro:sensor>
     <xacro:sensor parent="$(arg robot_name)_link_2" child="sensor_2_back">
@@ -26,5 +26,5 @@
     </xacro:sensor>
     <xacro:sensor parent="$(arg robot_name)_link_2" child="sensor_2_right">
-        <origin xyz="0 0.20 0.08" rpy="0 ${-PI / 2} ${-PI / 2}" />
+        <origin xyz="0 0.20 -0.08" rpy="0 ${PI / 2} ${PI / 2}" />
     </xacro:sensor>
     <xacro:sensor parent="$(arg robot_name)_link_4" child="sensor_4_front">
@@ -41,8 +41,8 @@
     </xacro:sensor>
     <xacro:sensor parent="$(arg robot_name)_link_6" child="sensor_6_front_left">
-        <origin xyz="-0.05 0.075 0.025" rpy="${PI / 180 * 87.5} ${PI / 180 * 45} ${PI / 180 * 175}" />
+        <origin xyz="-0.035 0.075 0.115" rpy="${PI / 180 * 93.5} ${PI / 180 * -50} ${PI / 180 * 175}" />
     </xacro:sensor>
     <xacro:sensor parent="$(arg robot_name)_link_6" child="sensor_6_front_right">
-        <origin xyz="-0.035 0.075 0.115" rpy="${PI / 180 * 93.5} ${PI / 180 * -50} ${PI / 180 * 175}" />
+        <origin xyz="-0.05 0.075 0.025" rpy="${PI / 180 * 87.5} ${PI / 180 * 45} ${PI / 180 * 175}" />
     </xacro:sensor>
     <!-- TODO: add tool here -->

Commit message: updated description of robot to better know about it's environment

File: iiwa_workcell_description/robots/iiwa_workcell.urdf.xacro (robot description, xacro)
@@ -8,9 +8,74 @@
     <xacro:arg name="origin_xyz" default="0 0 0" />
     <xacro:arg name="origin_rpy" default="0 0 0" />
-    <!-- Fix to world (we ignore the table the robot is mounted on for now) -->
-    <link name="world" />
-    <!-- TODO: add base here -->
+    <!-- world -->
+    <link name="world"/>
+    <!-- table -->
+    <joint name="world__table_joint" type="fixed">
+        <origin xyz="0 0 0.92" rpy="0 0 0"/>
+        <parent link="world"/>
+        <child link="table"/>
+    </joint>
+    <link name="table">
+        <visual>
+            <origin xyz="0 0 -${0.92 / 2}" rpy="0 0 0"/>
+            <geometry>
+                <box size="1.2 1.2 0.92"/>
+            </geometry>
+            <material name="Grey"/>
+        </visual>
+        <collision>
+            <origin xyz="0 0 -${0.92 / 2}" rpy="0 0 0"/>
+            <geometry>
+                <box size="1.2 1.2 0.92"/>
+            </geometry>
+            <material name="Grey"/>
+        </collision>
+    </link>
+    <!-- base -->
+    <joint name="table__base_joint" type="fixed">
+        <origin xyz="${(-1.2 + 0.245) / 2 + 0.225} ${(-1.2 + 0.245) / 2 + 0.327} 0.003" rpy="0 0 0"/>
+        <parent link="table"/>
+        <child link="base"/>
+    </joint>
+    <link name="base">
+        <visual>
+            <origin xyz="0 0 -${0.003 / 2}" rpy="0 0 0"/>
+            <geometry>
+                <box size="0.245 0.245 0.003"/>
+            </geometry>
+            <material name="Grey"/>
+        </visual>
+        <collision>
+            <origin xyz="0 0 -${0.003 / 2}" rpy="0 0 0"/>
+            <geometry>
+                <box size="0.245 0.245 0.003"/>
+            </geometry>
+            <material name="Grey"/>
+        </collision>
+    </link>
+    <!-- wall (to prevent accidental collision with adjacent robot) -->
+    <joint name="world__wall_joint" type="fixed">
+        <origin xyz="0 -0.65 1.5" rpy="0 0 0"/>
+        <parent link="world"/>
+        <child link="wall"/>
+    </joint>
+    <link name="wall">
+        <visual>
+            <origin xyz="0 0 0" rpy="0 0 0"/>
+            <geometry>
+                <box size="1.2 0.1 3"/>
+            </geometry>
+            <material name="Grey"/>
+        </visual>
+        <collision>
+            <origin xyz="0 0 0" rpy="0 0 0"/>
+            <geometry>
+                <box size="1.2 0.1 3"/>
+            </geometry>
+            <material name="Grey"/>
+        </collision>
+    </link>
     <!-- iiwa -->
-    <xacro:iiwa7 hardware_interface="$(arg hardware_interface)" robot_name="$(arg robot_name)" parent="world">
+    <xacro:iiwa7 hardware_interface="$(arg hardware_interface)" robot_name="$(arg robot_name)" parent="base">
         <origin xyz="$(arg origin_xyz)" rpy="$(arg origin_rpy)" />
     </xacro:iiwa7>
@@ -46,4 +111,25 @@
         <origin xyz="-0.05 0.075 0.025" rpy="${PI / 180 * 87.5} ${PI / 180 * 45} ${PI / 180 * 175}" />
     </xacro:sensor>
-    <!-- TODO: add tool here -->
+    <!-- tool -->
+    <joint name="$(arg robot_name)_link_ee__tool_joint" type="fixed">
+        <origin xyz="0 0 0" rpy="0 0 0"/>
+        <parent link="$(arg robot_name)_link_ee"/>
+        <child link="tool"/>
+    </joint>
+    <link name="tool">
+        <visual>
+            <origin xyz="0 0 0.075" rpy="0 0 0"/>
+            <geometry>
+                <cylinder radius="0.065" length="0.15"/>
+            </geometry>
+            <material name="Grey"/>
+        </visual>
+        <collision>
+            <origin xyz="0 0 0.075" rpy="0 0 0"/>
+            <geometry>
+                <cylinder radius="0.065" length="0.15"/>
+            </geometry>
+            <material name="Grey"/>
+        </collision>
+    </link>
 </robot>
